File: hardware/solderable_breadboard_mini.sch (EAGLE design)
At the start: 37 parts

Commit message: Adding some flame logos to the board.
Parts:
- added LOGO3, LOGO4: SFE_LOGO_FLAME.1_INCH, SparkFun-Aesthetics:SFE_LOGO_FLAME.1_INCH
Changed lines of the file:
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@@
 <part name="LOGO1" library="SparkFun-Aesthetics" deviceset="SFE_LOGO_NAME" device=".1_INCH"/>
 <part name="LOGO2" library="SparkFun-Aesthetics" deviceset="OSHW-LOGO" device="M"/>
+<part name="LOGO3" library="SparkFun-Aesthetics" deviceset="SFE_LOGO_FLAME" device=".1_INCH"/>
+<part name="LOGO4" library="SparkFun-Aesthetics" deviceset="SFE_LOGO_FLAME" device=".1_INCH"/>
 </parts>
 <sheets>
@@
 <instance part="LOGO1" gate="G$1" x="86.36" y="2.54"/>
 <instance part="LOGO2" gate="G$1" x="233.68" y="48.26"/>
+<instance part="LOGO3" gate="G$1" x="213.36" y="40.64"/>
+<instance part="LOGO4" gate="G$1" x="213.36" y="40.64"/>
 </instances>
 <busses>
